Commit message: Object avoidance (One sided)

File: src/lazysim/description/control.xacro (robot description, xacro)
@@ -5,4 +5,20 @@
             <plugin>gazebo_ros2_control/GazeboSystem</plugin>
         </hardware>
+        <joint name="base_to_front_left_hinge">
+            <command_interface name="position" />
+            <state_interface name="position" />
+        </joint>
+        <joint name="base_to_front_right_hinge">
+            <command_interface name="position" />
+            <state_interface name="position" />
+        </joint>
+        <joint name="front_left_hinge_to_wheel">
+            <command_interface name="velocity" />
+            <state_interface name="velocity" />
+        </joint>
+        <joint name="front_right_hinge_to_wheel">
+            <command_interface name="velocity" />
+            <state_interface name="velocity" />
+        </joint>
         <joint name="base_to_back_left_wheel">
             <command_interface name="velocity" />
@@ -13,13 +29,41 @@
             <state_interface name="velocity" />
         </joint>
+    </ros2_control>
+    <transmission name="front_left_steering_trans">
+        <type>transmission_interface/SimpleTransmission</type>
+        <actuator name="front_left_steer">
+            <mechanicalReduction>1.0</mechanicalReduction>
+        </actuator>
         <joint name="base_to_front_left_hinge">
-            <command_interface name="position" />
-            <state_interface name="position" />
+            <hardwareInterface>position</hardwareInterface>
         </joint>
+    </transmission>
+    <transmission name="front_right_steering_trans">
+        <type>transmission_interface/SimpleTransmission</type>
+        <actuator name="front_right_steer">
+            <mechanicalReduction>1.0</mechanicalReduction>
+        </actuator>
         <joint name="base_to_front_right_hinge">
-            <command_interface name="position" />
-            <state_interface name="position" />
+            <hardwareInterface>position</hardwareInterface>
         </joint>
-    </ros2_control>
+    </transmission>
+    <transmission name="front_left_wheel_trans">
+        <type>transmission_interface/SimpleTransmission</type>
+        <actuator name="front_left_wheel_motor">
+            <mechanicalReduction>1.0</mechanicalReduction>
+        </actuator>
+        <joint name="front_left_hinge_to_wheel">
+            <hardwareInterface>velocity</hardwareInterface>
+        </joint>
+    </transmission>
+    <transmission name="front_right_wheel_trans">
+        <type>transmission_interface/SimpleTransmission</type>
+        <actuator name="front_right_wheel_motor">
+            <mechanicalReduction>1.0</mechanicalReduction>
+        </actuator>
+        <joint name="front_right_hinge_to_wheel">
+            <hardwareInterface>velocity</hardwareInterface>
+        </joint>
+    </transmission>
     <transmission name="left_wheel_trans">
         <type>transmission_interface/SimpleTransmission</type>
@@ -28,5 +72,4 @@
         </actuator>
         <joint name="base_to_back_left_wheel">
-            <!-- <hardwareInterface>hardware_interface/VelocityJointInterface</hardwareInterface> -->
             <hardwareInterface>velocity</hardwareInterface>
         </joint>
@@ -38,26 +81,5 @@
         </actuator>
         <joint name="base_to_back_right_wheel">
-            <!-- <hardwareInterface>hardware_interface/VelocityJointInterface</hardwareInterface> -->
             <hardwareInterface>velocity</hardwareInterface>
-        </joint>
-    </transmission>
-    <transmission name="front_left_steering_trans">
-        <type>transmission_interface/SimpleTransmission</type>
-        <actuator name="front_left_steer">
-            <mechanicalReduction>1.0</mechanicalReduction>
-        </actuator>
-        <joint name="base_to_front_left_hinge">
-            <!-- <hardwareInterface>hardware_interface/PositionJointInterface</hardwareInterface> -->
-            <hardwareInterface>position</hardwareInterface>
-        </joint>
-    </transmission>
-    <transmission name="front_right_steering_trans">
-        <type>transmission_interface/SimpleTransmission</type>
-        <actuator name="front_right_steer">
-            <mechanicalReduction>1.0</mechanicalReduction>
-        </actuator>
-        <joint name="base_to_front_right_hinge">
-            <!-- <hardwareInterface>hardware_interface/PositionJointInterface</hardwareInterface> -->
-            <hardwareInterface>position</hardwareInterface>
         </joint>
     </transmission>
