Commit message: Odom Calculation

File: src/lazysim/description/lazyBot.xacro (robot description, xacro)
@@ -1,7 +1,31 @@
 <?xml version="1.0"?>
 <robot xmlns:xacro="http://www.ros.org/wiki/xacro" name="lazyBot">
+    <xacro:property name="wheelbase" value="0.12" />
+    <xacro:property name="len_offs" value="0.035" />
+    <xacro:property name="length" value="0.2" />
+    <xacro:property name="width" value="0.1" />
+    <xacro:property name="hinge_d" value="0.035" />
+    <xacro:property name="wheel_width" value="0.094" />
+    <xacro:property name="height" value="0.07" />
+    <xacro:property name="ground_offset" value="0.006" />
+    <xacro:property name="wheel_radius" value="0.02" />
+    <xacro:property name="wheel_length" value="0.005" />
+    <xacro:property name="laser_distance_from_base" value="0.09" />
+    <xacro:property name="laser_height" value="0.015" />
+    <xacro:property name="laser_radius" value="0.025" />
+    <xacro:property name="imu_distance_from_base" value="0.02" />
+    <xacro:property name="imu_size" value="0.02" />
+    <xacro:property name="camera_distance" value="0.15" />
+    <xacro:property name="camera_height" value="0.05" />
+    <xacro:property name="car_name" value="lazyBot" />
+    <xacro:property name="base_mass" value="1.5" />
+    <xacro:property name="wheel_mass" value="0.05" />
+    <xacro:property name="imu_mass" value="0.01" />
+    <xacro:property name="laser_mass" value="0.05" />
+    <xacro:property name="hinge_mass" value="0.01" />
     <xacro:include filename="lazyBotCore.xacro" />
     <xacro:include filename="lidar.xacro" />
     <xacro:include filename="camera.xacro" />
+    <xacro:include filename="IMU.xacro" />
     <xacro:include filename="gazebo.xacro" />
     <xacro:include filename="control.xacro" />

File: src/lazysim/description/lazyBotCore.xacro (robot description, xacro)
@@ -1,24 +1,4 @@
 <?xml version="1.0"?>
 <robot xmlns:xacro="http://www.ros.org/wiki/xacro" name="lazyBot">
-    <xacro:property name="wheelbase" value="0.12" />
-    <xacro:property name="len_offs" value="0.035" />
-    <xacro:property name="length" value="0.2" />
-    <xacro:property name="width" value="0.1" />
-    <xacro:property name="hinge_d" value="0.035" />
-    <xacro:property name="wheel_width" value="0.094" />
-    <xacro:property name="height" value="0.07" />
-    <xacro:property name="ground_offset" value="0.006" />
-    <xacro:property name="wheel_radius" value="0.02" />
-    <xacro:property name="wheel_length" value="0.005" />
-    <xacro:property name="laser_distance_from_base" value="0.09" />
-    <xacro:property name="laser_height" value="0.015" />
-    <xacro:property name="laser_radius" value="0.025" />
-    <xacro:property name="camera_distance" value="0.15" />
-    <xacro:property name="camera_height" value="0.05" />
-    <xacro:property name="car_name" value="lazyBot" />
-    <xacro:property name="base_mass" value="1.5" />
-    <xacro:property name="wheel_mass" value="0.05" />
-    <xacro:property name="laser_mass" value="0.05" />
-    <xacro:property name="hinge_mass" value="0.01" />
     <material name="black">
         <color rgba="0.2 0.2 0.2 1." />
