Commit message: Changed track creator parameters to yaml fixed bugs in the logic of lap counting

File: src/lazysim/description/IMU.xacro (robot description, xacro)
@@ -4,26 +4,13 @@
         <parent link="chassis" />
         <child link="imu" />
-        <origin xyz="${imu_distance_from_base} 0 ${ground_offset+height+(imu_size/2)}" />
+        <origin xyz="${imu_distance_from_base} 0 ${ground_offset+height+(imu_size/4)}" />
     </joint>
     <link name="imu">
         <visual>
             <geometry>
-                <box size="${imu_size} ${imu_size} ${imu_size}" />
+                <box size="${imu_size} ${imu_size} ${imu_size/2}" />
             </geometry>
             <material name="black" />
         </visual>
-        <collision self_collide="false">
-            <geometry>
-                <box size="${imu_size} ${imu_size} ${imu_size}" />
-            </geometry>
-        </collision>
-        <inertial>
-            <mass value="${imu_mass}" />
-            <inertia
-                ixx="${imu_mass/12 * (imu_size*imu_size + imu_size*imu_size)}"
-                iyy="${imu_mass/12 * (imu_size*imu_size + imu_size*imu_size)}"
-                izz="${imu_mass/12 * (imu_size*imu_size + imu_size*imu_size)}"
-                ixy="0" ixz="0" iyz="0" />
-        </inertial>
     </link>
     <gazebo reference="imu">

File: src/lazysim/description/lazyBot.xacro (robot description, xacro)
@@ -16,4 +16,5 @@
     <xacro:property name="imu_distance_from_base" value="0.02" />
     <xacro:property name="imu_size" value="0.02" />
+    <xacro:property name="proximity_size" value="0.01" />
     <xacro:property name="camera_distance" value="0.15" />
     <xacro:property name="camera_height" value="0.05" />
@@ -26,4 +27,5 @@
     <xacro:include filename="lazyBotCore.xacro" />
     <xacro:include filename="lidar.xacro" />
+    <xacro:include filename="proximity.xacro" />
     <xacro:include filename="camera.xacro" />
     <xacro:include filename="IMU.xacro" />

File: src/lazysim/description/lidar.xacro (robot description, xacro)
@@ -37,6 +37,6 @@
                     <horizontal>
                         <samples>720</samples>
-                        <min_angle>-3.14</min_angle>
-                        <max_angle>3.14</max_angle>
+                        <min_angle>${-pi}</min_angle>
+                        <max_angle>${pi}</max_angle>
                     </horizontal>
                 </scan>
