Commit message: Object detection with lidar

File: src/lazysim/description/lazyBotCore.xacro (robot description, xacro)
@@ -17,8 +17,8 @@
     <xacro:property name="camera_height" value="0.05" />
     <xacro:property name="car_name" value="lazyBot" />
-    <xacro:property name="base_mass" value="2.0" />
-    <xacro:property name="wheel_mass" value="0.1" />
-    <xacro:property name="laser_mass" value="0.2" />
-    <xacro:property name="hinge_mass" value="0.05" />
+    <xacro:property name="base_mass" value="1.5" />
+    <xacro:property name="wheel_mass" value="0.05" />
+    <xacro:property name="laser_mass" value="0.05" />
+    <xacro:property name="hinge_mass" value="0.01" />
     <material name="black">
         <color rgba="0.2 0.2 0.2 1." />
@@ -45,4 +45,12 @@
                 </geometry>
                 <origin rpy="0 0 0" />
+                <surface>
+                    <friction>
+                        <ode>
+                            <mu>1.0</mu>
+                            <mu2>1.0</mu2>
+                        </ode>
+                    </friction>
+                </surface>
             </collision>
             <inertial>

File: src/lazysim/description/lidar.xacro (robot description, xacro)
@@ -52,4 +52,7 @@
                 <output_type>sensor_msgs/LaserScan</output_type>
                 <frame_name>laser</frame_name>
+                <laserRetro>1.0</laserRetro>
+                <min_intensity>0.2</min_intensity>
+                <max_intensity>1.0</max_intensity>
             </plugin>
         </sensor>

Commit message: Added odometry to rviz

File: src/lazysim/description/lazyBotCore.xacro (robot description, xacro)
@@ -45,17 +45,11 @@
         </link>
     </xacro:macro>
-    <!-- <link name="base_footprint">
-    </link> -->
-    <!-- BASE LINK -->
-    <link name="base_link">
-    </link>
-    <!-- BASE_FOOTPRINT LINK -->
-    <joint name="base_footprint_joint" type="fixed">
-        <parent link="base_link"/>
-        <child link="base_footprint"/>
+    <!-- <joint name="base_footprint_joint" type="fixed">
+        <parent link="base_footprint"/>
+        <child link="base_link"/>
         <origin xyz="0 0 0" rpy="0 0 0"/>
     </joint>
-    <link name="base_footprint">
-    </link>
+    <link name="base_footprint"> </link> -->
+    <link name="base_link"> </link>
     <link name="chassis">
         <visual>
@@ -142,17 +136,3 @@
     </joint>
     <xacro:wheel_link name="front_right_wheel" radius="${wheel_radius}" length="${wheel_length}" mass="${wheel_mass}" />
-    <link name="steering_wheel">
-        <inertial>
-            <mass value="${hinge_mass}" />
-            <inertia ixx="${hinge_mass*0.01}" iyy="${hinge_mass*0.01}" izz="${hinge_mass*0.01}"
-                ixy="0" ixz="0" iyz="0" />
-        </inertial>
-    </link>
-    <joint name="steering_joint" type="revolute">
-        <parent link="chassis" />
-        <child link="steering_wheel" />
-        <origin xyz="0 ${length/2} ${height}" rpy="0 0 0" />
-        <axis xyz="1 0 0" />
-        <limit lower="${-pi/2}" upper="${pi/2}" effort="10" velocity="50" />
-    </joint>
 </robot>
