Commit message: simulation camera update

File: src/lazysim/description/camera.xacro (robot description, xacro)
@@ -1,8 +1,22 @@
 <?xml version="1.0"?>
 <robot xmlns:xacro="http://www.ros.org/wiki/xacro" >
+    <joint name="chassis_to_cam_servo" type="revolute">
+        <parent link="chassis" />
+        <child link="cam_servo_link" />
+        <origin xyz="${camera_distance} 0 ${camera_height}" />
+        <axis xyz="0 0 1" />
+        <limit lower="${-pi/2}" upper="${pi/2}" effort="10" velocity="50" />
+    </joint>
+    <link name="cam_servo_link">
+        <inertial>
+            <mass value="${hinge_mass}" />
+            <inertia ixx="${hinge_mass*0.01}" iyy="${hinge_mass*0.01}" izz="${hinge_mass*0.01}"
+                ixy="0" ixz="0" iyz="0" />
+        </inertial>
+    </link>
     <joint name="camera_joint" type="fixed">
-        <parent link="chassis"/>
+        <parent link="cam_servo_link"/>
         <child link="camera_link"/>
-        <origin xyz="${camera_distance} 0 ${camera_height}" rpy="0 0 0"/>
+        <origin xyz="0 0 0" rpy="0 ${pi/24} 0"/>
     </joint>
     <link name="camera_link">
@@ -28,5 +42,5 @@
             <camera>
                 <!-- <horizontal_fov>2.7925268</horizontal_fov> -->
-                <horizontal_fov>2.0944</horizontal_fov>
+                <horizontal_fov>${pi/3}</horizontal_fov>
                 <image>
                     <format>R8G8B8</format>

File: src/lazysim/description/control.xacro (robot description, xacro)
@@ -5,4 +5,8 @@
             <plugin>gazebo_ros2_control/GazeboSystem</plugin>
         </hardware>
+        <joint name="chassis_to_cam_servo">
+            <command_interface name="position" />
+            <state_interface name="position" />
+        </joint>
         <joint name="base_to_front_left_hinge">
             <command_interface name="position" />
@@ -34,4 +38,13 @@
         </joint>
     </ros2_control>
+    <transmission name="chassis_to_cam_servo_trans">
+        <type>transmission_interface/SimpleTransmission</type>
+        <actuator name="chassis_to_cam_servo_actuator">
+            <mechanicalReduction>1.0</mechanicalReduction>
+        </actuator>
+        <joint name="chassis_to_cam_servo">
+            <hardwareInterface>position</hardwareInterface>
+        </joint>
+    </transmission>
     <transmission name="front_left_steering_trans">
         <type>transmission_interface/SimpleTransmission</type>

File: src/lazysim/description/lazyBot.xacro (robot description, xacro)
@@ -18,5 +18,5 @@
     <xacro:property name="proximity_size" value="0.01" />
     <xacro:property name="camera_distance" value="0.15" />
-    <xacro:property name="camera_height" value="0.05" />
+    <xacro:property name="camera_height" value="0.12" />
     <xacro:property name="car_name" value="lazyBot" />
     <xacro:property name="base_mass" value="1.5" />
